Commit message: Simulation v1

File: URDFs/disc_blue.urdf (robot description, URDF)
Before this commit: robot disc, 1 links, 0 joints
Links:
- link base_link: geometry collision cylinder length=0.005 radius=0.007; visual cylinder length=0.005 radius=0.007

File: URDFs/disc_green.urdf (robot description, URDF)
Before this commit: robot disc, 1 links, 0 joints
Links:
- link base_link: geometry collision cylinder length=0.005 radius=0.007; visual cylinder length=0.005 radius=0.007

File: URDFs/disc_light_green.urdf (robot description, URDF)
Before this commit: robot disc, 1 links, 0 joints
Links:
- link base_link: geometry collision cylinder length=0.005 radius=0.007; visual cylinder length=0.005 radius=0.007

File: URDFs/disc_orange.urdf (robot description, URDF)
Before this commit: robot disc, 1 links, 0 joints
Links:
- link base_link: geometry collision cylinder length=0.005 radius=0.007; visual cylinder length=0.005 radius=0.007

File: URDFs/disc_red.urdf (robot description, URDF)
Before this commit: robot disc, 1 links, 0 joints
Links:
- link base_link: geometry collision cylinder length=0.005 radius=0.007; visual cylinder length=0.005 radius=0.007

File: URDFs/disc_yellow.urdf (robot description, URDF)
Before this commit: robot disc, 1 links, 0 joints
Links:
- link base_link: geometry collision cylinder length=0.005 radius=0.007; visual cylinder length=0.005 radius=0.007

File: URDFs/knife.urdf (robot description, URDF)
Before this commit: robot knife, 1 links, 0 joints
Links:
- link base_link: mass 0.4 -> 0.5; geometry collision box size=0.005 0.2 0.03; visual box size=0.005 0.2 0.03

Commit message: Image Processing

File: URDFs/disc_blue.urdf (robot description, URDF)
Before this commit: robot disc, 1 links, 0 joints
Links:
- link base_link: geometry collision cylinder length=0.005 radius=0.0035; visual cylinder length=0.005 radius=0.0035

File: URDFs/disc_green.urdf (robot description, URDF)
Before this commit: robot disc, 1 links, 0 joints
Links:
- link base_link: geometry collision cylinder length=0.005 radius=0.0035; visual cylinder length=0.005 radius=0.0035

File: URDFs/disc_light_green.urdf (robot description, URDF)
Before this commit: robot disc, 1 links, 0 joints
Links:
- link base_link: geometry collision cylinder length=0.005 radius=0.0035; visual cylinder length=0.005 radius=0.0035

File: URDFs/disc_orange.urdf (robot description, URDF)
Before this commit: robot disc, 1 links, 0 joints
Links:
- link base_link: geometry collision cylinder length=0.005 radius=0.0035; visual cylinder length=0.005 radius=0.0035

File: URDFs/disc_red.urdf (robot description, URDF)
Before this commit: robot disc, 1 links, 0 joints
Links:
- link base_link: geometry collision cylinder length=0.005 radius=0.0035; visual cylinder length=0.005 radius=0.0035

File: URDFs/disc_yellow.urdf (robot description, URDF)
Before this commit: robot disc, 1 links, 0 joints
Links:
- link base_link: geometry collision cylinder length=0.005 radius=0.0035; visual cylinder length=0.005 radius=0.0035
