Commit message: buggy lyapunov

File: URDFs/Assem2/urdf/Assem2.urdf (robot description, URDF)
Before this commit: robot Assem1, 1 links, 0 joints
Links:
- link base_link: mass 7.05107809575261 -> 7.0511; geometry collision mesh filename=package://Assem2/meshes/base_link.STL; visual mesh filename=package://Assem2/meshes/base_link.STL
