Commit message: buggy lyapunov

File: URDFs/Assem4/urdf/Assem4.urdf (robot description, URDF)
Before this commit: robot Assem2, 1 links, 0 joints
Links:
- link base_link: geometry collision mesh filename=package://Assem4/meshes/base_link.STL; visual mesh filename=package://Assem4/meshes/base_link.STL
