Commit message: buggy lyapunov

File: assets/franka_description/robots/franka_panda.urdf (robot description, URDF)
Before this commit: robot panda, 10 links, 9 joints
Links:
- link knife: mass 0.5 -> 0.9; geometry collision box size=0.003 0.1 0.03; visual box size=0.003 0.1 0.03
Joints:
- joint panda_hand_knife_joint: origin xyz=0.10 0 0.08 rpy=0 0 1.57079 -> xyz=0 0 0.08 rpy=0 0 1.57079

Commit message: video output

File: assets/franka_description/robots/franka_panda.urdf (robot description, URDF)
Before this commit: robot panda, 10 links, 9 joints
Joints:
- joint panda_hand_knife_joint: origin xyz=0 0 0.08 rpy=0 0 1.57079 -> xyz=0 0 0.08 rpy=0 0 0

Commit message: Simulator Working v1

File: assets/franka_description/robots/franka_panda.urdf (robot description, URDF)
Before this commit: robot panda, 10 links, 9 joints
Links:
- link knife: geometry collision box size=0.003 0.152 0.03; visual box size=0.003 0.152 0.03
